Commit message: 。

File: src/rokae_xmate3_ros2/urdf/xMate3.ros2_control.xacro (robot description, xacro)
@@ -11,4 +11,5 @@
         <state_interface name="position"/>
         <state_interface name="velocity"/>
+        <state_interface name="effort"/>
       </joint>
       <joint name="xmate_joint_2">
@@ -16,4 +17,5 @@
         <state_interface name="position"/>
         <state_interface name="velocity"/>
+        <state_interface name="effort"/>
       </joint>
       <joint name="xmate_joint_3">
@@ -21,4 +23,5 @@
         <state_interface name="position"/>
         <state_interface name="velocity"/>
+        <state_interface name="effort"/>
       </joint>
       <joint name="xmate_joint_4">
@@ -26,4 +29,5 @@
         <state_interface name="position"/>
         <state_interface name="velocity"/>
+        <state_interface name="effort"/>
       </joint>
       <joint name="xmate_joint_5">
@@ -31,4 +35,5 @@
         <state_interface name="position"/>
         <state_interface name="velocity"/>
+        <state_interface name="effort"/>
       </joint>
       <joint name="xmate_joint_6">
@@ -36,6 +41,12 @@
         <state_interface name="position"/>
         <state_interface name="velocity"/>
+        <state_interface name="effort"/>
       </joint>
     </ros2_control>
+    <gazebo>
+      <plugin filename="libgazebo_ros2_control.so" name="gazebo_ros2_control">
+        <parameters>$(arg package_share)/config/ros2_control.yaml</parameters>
+      </plugin>
+    </gazebo>
   </xacro:macro>
 </robot>

File: src/rokae_xmate3_ros2/urdf/xMate3.xacro (robot description, xacro)
@@ -1,8 +1,11 @@
 <?xml version="1.0" ?>
 <robot name="xMate3" xmlns:xacro="http://www.ros.org/wiki/xacro">
+  <xacro:include filename="xMate3.ros2_control.xacro"/>
   <!-- ==================== 常量定义 ==================== -->
   <xacro:property name="M_PI" value="3.1415926535897931"/>
   <xacro:property name="mesh_scale" value="0.001 0.001 0.001"/>
   <xacro:arg name="mesh_root" default="package://rokae_xmate3_ros2/models/rokae_xmate3_ros2/meshes/"/>
+  <xacro:arg name="package_share" default="."/>
+  <xacro:arg name="enable_ros2_control" default="false"/>
   <xacro:property name="mesh_prefix_root" value="$(arg mesh_root)"/>
   <xacro:property name="mesh_prefix_vis" value="${mesh_prefix_root}visual/"/>
@@ -60,14 +63,8 @@
   <!-- ==================== Transmission宏 ==================== -->
   <xacro:macro name="robot_transmission" params="name joint_name actuator_name">
-    <transmission name="${name}">
-      <type>transmission_interface/SimpleTransmission</type>
-      <joint name="${joint_name}">
-        <hardwareInterface>EffortJointInterface</hardwareInterface>
-      </joint>
-      <actuator name="${actuator_name}">
-        <hardwareInterface>EffortJointInterface</hardwareInterface>
-        <mechanicalReduction>1</mechanicalReduction>
-      </actuator>
-    </transmission>
+    <!-- Legacy transmissions are intentionally omitted in the ros2_control/Gazebo path.
+         The current simulation stack drives joints via ros2_control interfaces and the
+         xCore Gazebo plugin directly, so emitting ROS1-style transmissions only adds
+         redundant metadata and has been a frequent source of startup instability. -->
   </xacro:macro>
   <!-- ==================== 世界固定关节 ==================== -->
@@ -210,4 +207,7 @@
     <static>true</static>
   </gazebo>
+  <xacro:if value="$(arg enable_ros2_control)">
+    <xacro:xMate3_ros2_control/>
+  </xacro:if>
   <!-- xCore SDK 服务插件 - 直接控制关节，提供完整SDK功能 -->
   <gazebo>

Commit message: 。

File: src/rokae_xmate3_ros2/urdf/xMate3.ros2_control.xacro (robot description, xacro)
@@ -2,5 +2,8 @@
 <robot xmlns:xacro="http://www.ros.org/wiki/xacro">
   <!-- ==================== ROS2 Control 宏 ==================== -->
-  <xacro:macro name="xMate3_ros2_control" params="name:=xMate3_ros2_control">
+  <xacro:macro name="xMate3_ros2_control" params="name:=xMate3_ros2_control package_share:=. backend_mode:=jtc">
+    <xacro:property
+      name="ros2_control_config"
+      value="${str(package_share) + '/config/' + ('ros2_control_rt.yaml' if str(backend_mode) == 'hybrid' else 'ros2_control_nrt.yaml')}"/>
     <ros2_control name="${name}" type="system">
       <hardware>
@@ -46,5 +49,5 @@
     <gazebo>
       <plugin filename="libgazebo_ros2_control.so" name="gazebo_ros2_control">
-        <parameters>$(arg package_share)/config/ros2_control.yaml</parameters>
+        <parameters>${ros2_control_config}</parameters>
       </plugin>
     </gazebo>

File: src/rokae_xmate3_ros2/urdf/xMate3.xacro (robot description, xacro)
@@ -253,5 +253,5 @@
   </gazebo>
   <xacro:if value="${str(ros2_control_enabled).lower() == 'true' and str(backend_mode_value) != 'effort'}">
-    <xacro:xMate3_ros2_control/>
+    <xacro:xMate3_ros2_control package_share="$(arg package_share)" backend_mode="$(arg backend_mode)"/>
   </xacro:if>
   <!-- xCore SDK 服务插件 - 直接控制关节，提供完整SDK功能 -->
