Commit message: 无mv

File: src/rokae_xmate3_ros2/urdf/xMate3.xacro (robot description, xacro)
@@ -4,6 +4,8 @@
   <xacro:property name="M_PI" value="3.1415926535897931"/>
   <xacro:property name="mesh_scale" value="0.001 0.001 0.001"/>
-  <xacro:property name="mesh_prefix_vis" value="package://rokae_xmate3_ros2/meshes/visual/"/>
-  <xacro:property name="mesh_prefix_col" value="package://rokae_xmate3_ros2/meshes/collision/"/>
+  <xacro:arg name="mesh_root" default="package://rokae_xmate3_ros2/models/rokae_xmate3_ros2/meshes/"/>
+  <xacro:property name="mesh_prefix_root" value="$(arg mesh_root)"/>
+  <xacro:property name="mesh_prefix_vis" value="${mesh_prefix_root}visual/"/>
+  <xacro:property name="mesh_prefix_col" value="${mesh_prefix_root}collision/"/>
   <!-- ==================== 材料定义 ==================== -->
   <xacro:macro name="material_color" params="name r g b">

Commit message: 。

File: src/rokae_xmate3_ros2/urdf/xMate3.xacro (robot description, xacro)
@@ -8,7 +8,12 @@
   <xacro:arg name="package_share" default="."/>
   <xacro:arg name="enable_ros2_control" default="false"/>
+  <xacro:arg name="enable_xcore_plugin" default="true"/>
+  <xacro:arg name="backend_mode" default="hybrid"/>
   <xacro:property name="mesh_prefix_root" value="$(arg mesh_root)"/>
   <xacro:property name="mesh_prefix_vis" value="${mesh_prefix_root}visual/"/>
   <xacro:property name="mesh_prefix_col" value="${mesh_prefix_root}collision/"/>
+  <xacro:property name="ros2_control_enabled" value="$(arg enable_ros2_control)"/>
+  <xacro:property name="xcore_plugin_enabled" value="$(arg enable_xcore_plugin)"/>
+  <xacro:property name="backend_mode_value" value="$(arg backend_mode)"/>
   <!-- ==================== 材料定义 ==================== -->
   <xacro:macro name="material_color" params="name r g b">
@@ -207,10 +212,14 @@
     <static>true</static>
   </gazebo>
-  <xacro:if value="$(arg enable_ros2_control)">
+  <xacro:if value="${str(ros2_control_enabled).lower() == 'true' and str(backend_mode_value) != 'effort'}">
     <xacro:xMate3_ros2_control/>
   </xacro:if>
   <!-- xCore SDK 服务插件 - 直接控制关节，提供完整SDK功能 -->
-  <gazebo>
-    <plugin name="xcore_controller_gazebo_plugin" filename="libxcore_controller_gazebo_plugin.so"/>
-  </gazebo>
+  <xacro:if value="${str(xcore_plugin_enabled).lower() == 'true' and str(backend_mode_value) != 'jtc'}">
+    <gazebo>
+      <plugin name="xcore_controller_gazebo_plugin" filename="libxcore_controller_gazebo_plugin.so">
+        <backend_mode>${backend_mode_value}</backend_mode>
+      </plugin>
+    </gazebo>
+  </xacro:if>
 </robot>

Commit message: .

File: src/rokae_xmate3_ros2/urdf/xMate3.xacro (robot description, xacro)
@@ -10,4 +10,10 @@
   <xacro:arg name="enable_xcore_plugin" default="true"/>
   <xacro:arg name="backend_mode" default="hybrid"/>
+  <xacro:arg name="joint_damping" default="0.5"/>
+  <xacro:arg name="joint_friction" default="0.1"/>
+  <xacro:arg name="flange_to_tool0_xyz" default="0 0 0"/>
+  <xacro:arg name="tool0_to_tcp_xyz" default="0 0 0"/>
+  <xacro:arg name="payload_xyz" default="0 0 0"/>
+  <xacro:arg name="payload_mass" default="0.0001"/>
   <xacro:property name="mesh_prefix_root" value="$(arg mesh_root)"/>
   <xacro:property name="mesh_prefix_vis" value="${mesh_prefix_root}visual/"/>
@@ -16,4 +22,6 @@
   <xacro:property name="xcore_plugin_enabled" value="$(arg enable_xcore_plugin)"/>
   <xacro:property name="backend_mode_value" value="$(arg backend_mode)"/>
+  <xacro:property name="joint_damping_value" value="$(arg joint_damping)"/>
+  <xacro:property name="joint_friction_value" value="$(arg joint_friction)"/>
   <!-- ==================== 材料定义 ==================== -->
   <xacro:macro name="material_color" params="name r g b">
@@ -55,5 +63,5 @@
   </xacro:macro>
   <!-- ==================== Joint宏 ==================== -->
-  <xacro:macro name="robot_joint" params="name parent child axis_x axis_y axis_z limit_effort limit_lower limit_upper limit_vel ox oy oz damping:=0.5">
+  <xacro:macro name="robot_joint" params="name parent child axis_x axis_y axis_z limit_effort limit_lower limit_upper limit_vel ox oy oz damping:=${joint_damping_value} friction:=${joint_friction_value}">
     <joint name="${name}" type="revolute">
       <parent link="${parent}"/>
@@ -62,7 +70,15 @@
       <axis xyz="${axis_x} ${axis_y} ${axis_z}"/>
       <origin rpy="0 0 0" xyz="${ox} ${oy} ${oz}"/>
-      <!-- 阻尼改为0.5，补充小摩擦提升稳定性 -->
-      <dynamics damping="${damping}" friction="0.1"/>
+      <dynamics damping="${damping}" friction="${friction}"/>
     </joint>
+  </xacro:macro>
+  <xacro:macro name="frame_link" params="name mass:=0.0001">
+    <link name="${name}">
+      <inertial>
+        <origin xyz="0 0 0" rpy="0 0 0"/>
+        <mass value="${mass}"/>
+        <inertia ixx="1e-6" ixy="0" ixz="0" iyy="1e-6" iyz="0" izz="1e-6"/>
+      </inertial>
+    </link>
   </xacro:macro>
   <!-- ==================== Transmission宏 ==================== -->
@@ -208,4 +224,28 @@
     ox="0" oy="0.017" oz="-0.043"
     vis_material="white"/>
+  <xacro:frame_link name="flange"/>
+  <joint name="xmate_flange_joint" type="fixed">
+    <parent link="xMate3_link6"/>
+    <child link="flange"/>
+    <origin xyz="0 0 0" rpy="0 0 0"/>
+  </joint>
+  <xacro:frame_link name="tool0"/>
+  <joint name="xmate_tool0_joint" type="fixed">
+    <parent link="flange"/>
+    <child link="tool0"/>
+    <origin xyz="$(arg flange_to_tool0_xyz)" rpy="0 0 0"/>
+  </joint>
+  <xacro:frame_link name="tcp"/>
+  <joint name="xmate_tcp_joint" type="fixed">
+    <parent link="tool0"/>
+    <child link="tcp"/>
+    <origin xyz="$(arg tool0_to_tcp_xyz)" rpy="0 0 0"/>
+  </joint>
+  <xacro:frame_link name="payload" mass="$(arg payload_mass)"/>
+  <joint name="xmate_payload_joint" type="fixed">
+    <parent link="tcp"/>
+    <child link="payload"/>
+    <origin xyz="$(arg payload_xyz)" rpy="0 0 0"/>
+  </joint>
   <!-- 强制锁定基座，Gazebo中不会被重力影响、不会移动 -->
   <gazebo reference="xMate3_base">

Commit message: 。

File: src/rokae_xmate3_ros2/urdf/xMate3.xacro (robot description, xacro)
@@ -7,7 +7,8 @@
   <xacro:arg name="mesh_root" default="package://rokae_xmate3_ros2/models/rokae_xmate3_ros2/meshes/"/>
   <xacro:arg name="package_share" default="."/>
-  <xacro:arg name="enable_ros2_control" default="false"/>
+  <xacro:arg name="enable_ros2_control" default="true"/>
   <xacro:arg name="enable_xcore_plugin" default="true"/>
-  <xacro:arg name="backend_mode" default="hybrid"/>
+  <xacro:arg name="backend_mode" default="jtc"/>
+  <xacro:arg name="service_exposure_profile" default="public_xmate6_only"/>
   <xacro:arg name="joint_damping" default="0.5"/>
   <xacro:arg name="joint_friction" default="0.1"/>
@@ -22,4 +23,5 @@
   <xacro:property name="xcore_plugin_enabled" value="$(arg enable_xcore_plugin)"/>
   <xacro:property name="backend_mode_value" value="$(arg backend_mode)"/>
+  <xacro:property name="service_exposure_profile_value" value="$(arg service_exposure_profile)"/>
   <xacro:property name="joint_damping_value" value="$(arg joint_damping)"/>
   <xacro:property name="joint_friction_value" value="$(arg joint_friction)"/>
@@ -255,9 +257,10 @@
     <xacro:xMate3_ros2_control package_share="$(arg package_share)" backend_mode="$(arg backend_mode)"/>
   </xacro:if>
-  <!-- xCore SDK 服务插件 - 直接控制关节，提供完整SDK功能 -->
-  <xacro:if value="${str(xcore_plugin_enabled).lower() == 'true' and str(backend_mode_value) != 'jtc'}">
+  <!-- xCore SDK 服务插件 - 提供 xCore SDK 兼容服务与 runtime，jtc 模式下仅让执行权保持在外部 JTC -->
+  <xacro:if value="${str(xcore_plugin_enabled).lower() == 'true'}">
     <gazebo>
       <plugin name="xcore_controller_gazebo_plugin" filename="libxcore_controller_gazebo_plugin.so">
         <backend_mode>${backend_mode_value}</backend_mode>
+        <service_exposure_profile>${service_exposure_profile_value}</service_exposure_profile>
       </plugin>
     </gazebo>

Commit message: 。

File: src/rokae_xmate3_ros2/urdf/xMate3.xacro (robot description, xacro)
@@ -10,5 +10,6 @@
   <xacro:arg name="enable_xcore_plugin" default="true"/>
   <xacro:arg name="backend_mode" default="jtc"/>
-  <xacro:arg name="service_exposure_profile" default="public_xmate6_only"/>
+  <xacro:arg name="service_exposure_profile" default="public_xmate_er3_only"/>
+  <xacro:arg name="compatibility_alias_policy" default="canonical_plus_compat"/>
   <xacro:arg name="joint_damping" default="0.5"/>
   <xacro:arg name="joint_friction" default="0.1"/>
@@ -24,4 +25,5 @@
   <xacro:property name="backend_mode_value" value="$(arg backend_mode)"/>
   <xacro:property name="service_exposure_profile_value" value="$(arg service_exposure_profile)"/>
+  <xacro:property name="compatibility_alias_policy_value" value="$(arg compatibility_alias_policy)"/>
   <xacro:property name="joint_damping_value" value="$(arg joint_damping)"/>
   <xacro:property name="joint_friction_value" value="$(arg joint_friction)"/>
@@ -263,4 +265,5 @@
         <backend_mode>${backend_mode_value}</backend_mode>
         <service_exposure_profile>${service_exposure_profile_value}</service_exposure_profile>
+        <compatibility_alias_policy>${compatibility_alias_policy_value}</compatibility_alias_policy>
       </plugin>
     </gazebo>
